File: kicad projet/hsensor/hsensor.kicad_sch (KiCad schematic)
At the start: 33 parts, among them J1 Conn_01x01_Socket, J12 BNC OUT, J2 Conn_01x01_Socket, J2_0 Conn_01x02_Pin, J2_1 Conn_01x02_Pin, J2_2 Conn_01x02_Pin, J3 Conn_01x03_Pin, U1 TLV75801PDBV, U2 TLV75801PDBV, U3 LM358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

Commit message: final pcb (i hope)
Parts:
- A1: footprint Module:RaspberryPi_Pico_W_SMD -> Module:RaspberryPi_Pico_Common_THT
- RV3: value 5e3 -> 5.e3; footprint Resistor_SMD:R_1206_3216Metric -> Potentiometer_THT:Potentiometer_Bourns_3266Y_Vertical
- U4: footprint TCRT5000:OPTO_TCRT5000 -> Sensor:OPTO_TCRT5000
